File: Cable-Test-RJ45-RJ12.brd (EAGLE design)
At the start: 86.7 x 32.6 mm, 28 parts, among them IC1 555, IC2 4017N, J2 RJ11, J4 RJ11, SW1 PB7-0

Commit message: Version 0.4
Version 0.4, I add a "C3" to stabilize the clock signal impulses
Parts:
- added C3: 0.1uF, capacitor-wima:C2.5-2
- C2: value 100nF -> 0.1uF
- moved C2 2.68 mm to (22.5, 30.7), turned to 180 degrees
Connections:
- net GND: now also C3.2
- net Q: now also C3.1
Routing:
- net Q: track 42.3 -> 53.8 mm
- net VCC: track 48.2 -> 53.6 mm, vias 0 -> 1
- net GND: track 5.29 -> 0.00 mm, vias 2 -> 4
Other:
- board text added: "2109"
- board text added: "CERN-OHL-W V2"
- board text added: "Rev.04"
- board text removed: "1919"

Commit message: Version 0.4
Parts:
- added D7: 1N4148, diode:D-2.5
- added D8: (no value), diode:D-2.5
- D4: value (none) -> 1N4148
- moved D4 58.8 mm to (26.6, 13.1), turned to 270 degrees
- moved R4 2.44 mm to (25.8, 6.21)
- moved D1 0.08 mm to (26.6, 26.5)
Connections:
- removed net N$3: D1.C, IC2.3, LB1.1
- new net N$6: IC2.3, LB1.1
- net 1: no longer D1.A
- net 2: now also D1.A
- net COMMON: now also D7.A, D8.A; no longer D4.A
- net N$13: now also D1.C
- net N$2: now also D6.C
- net N$20: no longer D6.C
- net N$23: now also D4.C
- net N$7: now also D8.C; no longer D4.C
- net N$8: now also D7.C
- net N$9: now also D4.A
Routing:
- net N$3: track 15.4 -> 0.00 mm
- net N$6: track 0.00 -> 15.3 mm
- net 2: track 48.6 -> 60.0 mm
- net 1: track 57.9 -> 46.6 mm
- net N$9: track 40.1 -> 48.9 mm
- net Q: track 53.8 -> 46.0 mm
- net N$8: track 26.8 -> 34.6 mm
- net N$17: track 43.1 -> 36.5 mm
- net N$20: track 29.7 -> 24.3 mm
- net N$2: track 28.5 -> 33.9 mm
- net N$28: track 15.5 -> 20.0 mm
- net 4: track 42.4 -> 45.1 mm, vias 0 -> 2
- net N$32: track 2.61 -> 4.49 mm
- net N$23: track 9.85 -> 11.1 mm
- net N$13: track 14.5 -> 15.6 mm
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Other:
- board text added: "CableTest"
- board text removed: "Cable test"
