File: Cable-Test-RJ45-RJ12.sch (EAGLE design)
At the start: 24 parts, among them IC1 555, IC2 4017N, J2 RJ11, J4 RJ11, SW1 PB7-0

Commit message: Version 0.4
Version 0.4, I add a "C3" to stabilize the clock signal impulses
Parts:
- added C3: 0.1uF, capacitor-wima:C2.5/2
- C2: value 100nF -> 0.1uF
Connections:
- net GND: now also C3.2
- net Q: now also C3.1
Other:
- note added: "04"
- note added: "CERN-OHL-W V2"
- moved on the sheet: LB1-10, R4

Commit message: Version 0.4
Parts:
- added D7: 1N4148, diode:DIODE-D-2.5
- added D8: (no value), diode:DIODE-D-2.5
- D4: value (none) -> 1N4148
Connections:
- removed net N$3: D1.C, IC2A.Q0, LB1-1.A
- new net N$6: IC2A.Q0, LB1-1.A
- net 1: no longer D1.A
- net 2: now also D1.A
- net COMMON: now also D7.A, D8.A; no longer D4.A
- net N$13: now also D1.C
- net N$2: now also D6.C
- net N$20: no longer D6.C
- net N$23: now also D4.C
- net N$7: now also D8.C; no longer D4.C
- net N$8: now also D7.C
- net N$9: now also D4.A
Other:
- moved on the sheet: D4, LB1-5, LB1-6, LB1-7, LB1-8, LB1-9
